Commit message: got planning in sim

File: src/main_computer_urc/description/robot.ros2_control.xacro (robot description, xacro)
@@ -38,4 +38,25 @@
         <state_interface name="position"/>
       </joint>
+      <joint name="${prefix}wrist1">
+        <command_interface name="position">
+          <param name="min">-1</param>
+          <param name="max">1</param>
+        </command_interface>
+        <state_interface name="position"/>
+      </joint>
+      <joint name="${prefix}wrist2_joint">
+        <command_interface name="position">
+          <param name="min">-1</param>
+          <param name="max">1</param>
+        </command_interface>
+        <state_interface name="position"/>
+      </joint>
+      <joint name="${prefix}wrist3_joint">
+        <command_interface name="position">
+          <param name="min">-1</param>
+          <param name="max">1</param>
+        </command_interface>
+        <state_interface name="position"/>
+      </joint>
     </ros2_control>
     <!-- <gazebo>
