Commit message: about to switch to velcoity control

File: src/main_computer_urc/description/robot-body.urdf.xacro (robot description, xacro)
@@ -12,4 +12,6 @@
   <!-- todo check axual offset for correctness -->
   <xacro:property name="axel_offset" value="0.025" /> <!-- Space btw top of beam and the each joint -->
+  <xacro:property name="damping" value="0.7" />
+  <xacro:property name="friction" value="50" />
   <joint name="${prefix}base_base" type="fixed">
     <xacro:insert_block name="origin" />
@@ -25,5 +27,6 @@
     <child link="${prefix}base_arm_link" />
     <axis xyz="0 0 1"/>
-    <dynamics damping="0.7"/>
+    <dynamics damping="${damping}"/>
+    <dynamics friction="${friction}"/>
     <limit effort="100" velocity="1.0"/>
   </joint>
@@ -57,5 +60,6 @@
     <origin xyz="0 0 ${height1}" rpy="0 0 0"/>
     <axis xyz="0 1 0"/>
-    <dynamics damping="0.7"/>
+    <dynamics damping="${damping}"/>
+    <dynamics friction="${friction}"/>
     <limit effort="100" velocity="1.0"/>
   </joint>
@@ -89,5 +93,6 @@
     <origin xyz="0 ${width} ${height2 - axel_offset*2}" rpy="0 0 0"/>
     <axis xyz="0 1 0"/>
-    <dynamics damping="0.7"/>
+    <dynamics damping="${damping}"/>
+    <dynamics friction="${friction}"/>
     <limit effort="100" velocity="1.0"/>
   </joint>
@@ -115,10 +120,10 @@
     </visual>
     <inertial>
-      <origin xyz="-0.00009299 0.031668 0.45103767" rpy="0 0 0"/>
-      <mass value="1.57816"/>
-      <inertia
-        ixx="0.029411" ixy="0.00000451" ixz="-0.00001344"
-        iyy="0.027431" iyz="-0.0031087"
-        izz="0.0026470"/>
+      <origin xyz="-0.00002531 -0.029129 0.38624" rpy="0 0 0"/>
+      <mass value="0.71617"/>
+      <inertia
+        ixx="0.0216357" ixy="-0.00000056" ixz="0.00000268"
+        iyy="0.021156" iyz="0.0015021"
+        izz="0.00060628"/>
     </inertial>
   </link>
@@ -155,5 +160,6 @@
     <origin xyz="0 ${wrist1AxelGap + width/2} ${height3 - axel_offset*2}" rpy="0 0 0"/>
     <axis xyz="0 1 0"/>
-    <dynamics damping="0.7"/>
+    <dynamics damping="${damping}"/>
+    <dynamics friction="${friction}"/>
     <limit effort="100" velocity="1.0"/>
   </joint>
@@ -172,12 +178,12 @@
       <material name="green"/>
     </visual>
-    <!-- <inertial>
-      <origin xyz="0 0 ${- height3/2 + axel_offset}" rpy="0 0 0"/>
-      <mass value="${mass}"/>
-      <inertia
-        ixx="${mass / 12.0 * (width*width + height3*height3)}" ixy="0.0" ixz="0.0"
-        iyy="${mass / 12.0 * (height3*height3 + width*width)}" iyz="0.0"
-        izz="${mass / 12.0 * (width*width + width*width)}"/>
-    </inertial> -->
+    <inertial>
+      <origin xyz="0.011680 0.024878 -0.0007064" rpy="0 0 0"/>
+      <mass value="0.49788"/>
+      <inertia
+        ixx="0.00014917" ixy="-0.00002443" ixz="0.00000086"
+        iyy="0.00050396" iyz="0.00000032"
+        izz="0.00053155"/>
+    </inertial>
   </link>
   <!-- Wrist 3 -->
@@ -194,5 +200,6 @@
     <origin xyz="${-wrist2AxelToRectTop} ${wrist2SizeY/2} ${0}" rpy="0 0 0"/>
     <axis xyz="1 0 0"/>
-    <dynamics damping="0.7"/>
+    <dynamics damping="${damping}"/>
+    <dynamics friction="${friction}"/>
     <limit effort="100" velocity="1.0"/>
   </joint>
@@ -219,4 +226,12 @@
         izz="${mass / 12.0 * (width*width + width*width)}"/>
     </inertial> -->
+    <inertial>
+      <origin xyz="-0.026878 -0.00007064 0.011680" rpy="0 0 0"/>
+      <mass value="0.49788"/>
+      <inertia
+        ixx="0.00050396" ixy="-0.00000032" ixz="-0.00002443"
+        iyy="0.00053155" iyz="-0.00000086"
+        izz="0.00014917"/>
+    </inertial>
   </link>
 <!-- end effector -->
@@ -233,5 +248,6 @@
     <origin xyz="${-wrist3SizeX/2} 0 ${0}" rpy="0 0 0"/>
     <axis xyz="0 0 1"/>
-    <dynamics damping="0.7"/>
+    <dynamics damping="${damping}"/>
+    <dynamics friction="${friction}"/>
     <limit effort="100" velocity="1.0"/>
   </joint>
@@ -250,12 +266,12 @@
       <material name="white"/>
     </visual>
-    <!-- <inertial>
-      <origin xyz="0 0 ${- height3/2 + axel_offset}" rpy="0 0 0"/>
-      <mass value="${mass}"/>
-      <inertia
-        ixx="${mass / 12.0 * (width*width + height3*height3)}" ixy="0.0" ixz="0.0"
-        iyy="${mass / 12.0 * (height3*height3 + width*width)}" iyz="0.0"
-        izz="${mass / 12.0 * (width*width + width*width)}"/>
-    </inertial> -->
+    <inertial>
+      <origin xyz="-0.038139 0.016827 -0.052402" rpy="0 0 0"/>
+      <mass value="0.59465"/>
+      <inertia
+        ixx="0.00061465" ixy="0.00023266" ixz="0.00017509"
+        iyy="0.00117167" iyz="-0.00007772"
+        izz="0.0011538"/>
+    </inertial>
   </link>
   <joint name="${prefix}tool_joint" type="fixed">

File: src/main_computer_urc/description/robot.ros2_control.xacro (robot description, xacro)
@@ -7,6 +7,6 @@
         <!-- <plugin>gz_ros2_control/GazeboSimSystem</plugin> -->
         <!-- By default, set up controllers for simulation. This won't work on real hardware -->
-        <plugin>mock_components/GenericSystem</plugin>
-        <!-- <plugin>main_computer_urc/MockArmHardware</plugin> -->
+        <!-- <plugin>mock_components/GenericSystem</plugin> -->
+        <plugin>main_computer_urc/MockArmHardware</plugin>
         <!-- </xacro:if> -->
         <!-- <xacro:unless value="${use_gazebo}">
@@ -18,5 +18,5 @@
       </hardware>
       <joint name="${prefix}base_joint">
-        <command_interface name="position">
+        <command_interface name="velocity">
           <param name="min">-1</param>
           <param name="max">1</param>
@@ -25,5 +25,5 @@
       </joint>
       <joint name="${prefix}shoulder">
-        <command_interface name="position">
+        <command_interface name="velocity">
           <param name="min">-1</param>
           <param name="max">1</param>
@@ -32,5 +32,5 @@
       </joint>
       <joint name="${prefix}elbow">
-        <command_interface name="position">
+        <command_interface name="velocity">
           <param name="min">-1</param>
           <param name="max">1</param>
@@ -41,5 +41,5 @@
       </joint>
       <joint name="${prefix}wrist1">
-        <command_interface name="position">
+        <command_interface name="velocity">
           <param name="min">-1</param>
           <param name="max">1</param>
@@ -48,5 +48,5 @@
       </joint>
       <joint name="${prefix}wrist2_joint">
-        <command_interface name="position">
+        <command_interface name="velocity">
           <param name="min">-1</param>
           <param name="max">1</param>
@@ -55,5 +55,5 @@
       </joint>
       <joint name="${prefix}wrist3_joint">
-        <command_interface name="position">
+        <command_interface name="velocity">
           <param name="min">-1</param>
           <param name="max">1</param>

Commit message: make PR fixes

File: src/main_computer_urc/description/robot-body.urdf.xacro (robot description, xacro)
@@ -10,5 +10,4 @@
   <xacro:property name="width" value="0.0254" /> <!-- Square dimensions (widthxwidth) of beams -->
   <xacro:property name="height3" value="0.5631" /> <!-- Link 3 -->
-  <!-- todo check axual offset for correctness -->
   <xacro:property name="axel_offset" value="0.025" /> <!-- Space btw top of beam and the each joint -->
   <xacro:property name="damping" value="0.7" />
@@ -112,9 +111,5 @@
       <geometry>
         <box size="${width} ${width} ${height3}"/>
-        <!-- <box size="${olnaextrasizex*5} ${olnaextra2sizey} ${olnaextra2sizez}" xyz="0 0 ${height3 - axel_offset}"/> -->
-      </geometry>
-      <!-- <geometry>
-        <box size="0.1 0.1 0.1"/>
-      </geometry> -->
+      </geometry>
       <material name="orange"/>
     </visual>
@@ -131,5 +126,4 @@
     <parent link="${prefix}link2"/>
     <child link="${prefix}link2_box"/>
-    <!-- <origin xyz="0 ${width} ${height2 - axel_offset*2}" rpy="0 0 0"/> -->
     <axis xyz="0 1 0"/>
   </joint>
@@ -218,12 +212,5 @@
       <material name="blue"/>
     </visual>
-    <!-- <inertial>
-      <origin xyz="0 0 ${- height3/2 + axel_offset}" rpy="0 0 0"/>
-      <mass value="${mass}"/>
-      <inertia
-        ixx="${mass / 12.0 * (width*width + height3*height3)}" ixy="0.0" ixz="0.0"
-        iyy="${mass / 12.0 * (height3*height3 + width*width)}" iyz="0.0"
-        izz="${mass / 12.0 * (width*width + width*width)}"/>
-    </inertial> -->
+    <!-- TODO URC-442: add in a mass and moment of inertia for Wrist3 -->
     <inertial>
       <origin xyz="-0.026878 -0.00007064 0.011680" rpy="0 0 0"/>

Commit message: Michael sar day 2025 (#21)
* lusi vision launched fine

* diff index cameras are working

* moveit-arm-stuff-squash

got a robot displaying with rviz and joint publisher gui

have arm elbow shoulder 2 link subset urdf

add basic movit config

update moveit package

trying to add gazebo

fix gazebo for michael's mackbook from crashing

working towards movit with ros2 control

wokring on getting ros2 control working

got past last ros2 control problem -- needed to remap expected robot description field

finally able to load the joint state publisher controller

working but going to reconfig moveit config

MOVIT PLAN EXECUTION WORKSgit status

WIP adding ros commanding node

still can't get new package to build

fix building of base station

broke drivline but have arm code module except for mock hardware interface

have a hardware plugin getting commands from moveit

publishing arm movements to topic

going to try testing on hardware

extra motor can more following path multiple times -- position is read back into trviz

got real arm moving to howdy

did work today -- now doing pid testing wiht real pos encoder from in motors

done with pid tunings that worked for big movements

updated tunings for movit keyframe

start impl tina feedback

Merge working driveline code to Michael's branch (#17)

* everything including driveline and arm compiled

* got further with driveline

* driveline code working

* add github action from main

* activate GitHub Action for a PR on any branch

* remove openCV build

* properly update dockerBuild

* fix the things

---------

Co-authored-by: Michael Baron <mike.init246@gmail.com>
Co-authored-by: Michael A. Baron <22025191+n4226@users.noreply.github.com>

adding base joint

base rot working

wrist one good

wrist 3 on arm

add endeff and collidors

got planning in sim

got 6 dof moving in simulation

start progress to get 6 joints in hardware working

arm preplanned moves workinggit add .git add .git add . all 6 axes

Merge in Tina's work on velocity control to get working on full arm (#18)

* Added moveit move group node

* everything to make boost disappear YAYYYYY

* launch armcommandencoder working

* ArmCommandEncoder is behaving fine

* there is a panda in my code

---------

Co-authored-by: Anders Heyniger <anders.heyniger@gmail.com>
Co-authored-by: Tina Pham <tip226@lehigh.edu>

switch to simulation and interial urdf removal for base

fix docker to not compule openCV

got moveit servo node to not crash with right config

servo moveit control working in sim

fixed some thigns in sim

debugging moveit servo on real arm last night

aruco tag working on mackbook pro

got lidar working -- main_comp launches with privliged to get camera working

pre tuesday testing

arm servo working in sim

servo still being weird but planning working well

post wedensday drew freed

ready try to fix Is

working

can't get sim servo to move

about to switch to velcoity control

got interactive marker working

* implimented end effector buttons???

* one lusi vision frame working????

* end effector minipulator in rviz and eend efect close open works on rover

* SAR submitted

* make PR fixes

---------

Co-authored-by: Tina Pham <tip226@lehigh.edu>

File: src/main_computer_urc/description/robot-body.urdf.xacro (robot description, xacro)
@@ -1,23 +1,39 @@
 <?xml version="1.0"?>
 <robot xmlns:xacro="http://www.ros.org/wiki/xacro">
-  <xacro:macro name="rrbot" params="parent prefix *origin">
+  <xacro:macro name="robot" params="parent prefix *origin">
   <!-- Constants for robot dimensions -->
-  <xacro:property name="mass" value="1" /> <!-- arbitrary value for mass -->
-  <xacro:property name="width" value="0.1" /> <!-- Square dimensions (widthxwidth) of beams -->
-  <xacro:property name="height1" value="0.1" /> <!-- Link 1 -->
-  <xacro:property name="height2" value="1" /> <!-- Link 2 -->
-  <xacro:property name="height3" value="1" /> <!-- Link 3 -->
-  <xacro:property name="axel_offset" value="0.05" /> <!-- Space btw top of beam and the each joint -->
-  <joint name="${prefix}base_joint" type="fixed">
+  <!-- <xacro:property name="mass" value="3" /> < arbitrary value for mass > -->
+  <xacro:property name="base_width" value="0.13" /> <!-- Square dimensions (widthxwidth) of beams -->
+  <xacro:property name="base_depth" value="0.102" /> <!-- Square dimensions (widthxwidth) of beams -->
+  <xacro:property name="height1" value="0.05" /> <!-- Link 1 -->
+  <xacro:property name="height2" value="0.5631" /> <!-- Link 2 -->
+  <xacro:property name="width" value="0.0254" /> <!-- Square dimensions (widthxwidth) of beams -->
+  <xacro:property name="height3" value="0.5631" /> <!-- Link 3 -->
+  <xacro:property name="axel_offset" value="0.025" /> <!-- Space btw top of beam and the each joint -->
+  <xacro:property name="damping" value="0.7" />
+  <xacro:property name="friction" value="50" />
+  <joint name="${prefix}base_base" type="fixed">
     <xacro:insert_block name="origin" />
     <parent link="${parent}"/>
     <child link="${prefix}base_link" />
+    <axis xyz="0 1 0"/>
+  </joint>
+  <link name="${prefix}base_link">
+  </link>
+<!--  shoulder motor -->
+  <joint name="${prefix}base_joint" type="continuous">
+    <parent link="${prefix}base_link"/>
+    <child link="${prefix}base_arm_link" />
+    <axis xyz="0 0 1"/>
+    <dynamics damping="${damping}"/>
+    <dynamics friction="${friction}"/>
+    <limit effort="100" velocity="1.0"/>
   </joint>
   <!-- Base Link -->
-  <link name="${prefix}base_link">
+  <link name="${prefix}base_arm_link">
     <collision>
       <origin xyz="0 0 ${height1/2}" rpy="0 0 0"/>
       <geometry>
-        <box size="${width} ${width} ${height1}"/>
+        <box size="${base_width} ${base_depth} ${height1}"/>
       </geometry>
     </collision>
@@ -25,9 +41,9 @@
       <origin xyz="0 0 ${height1/2}" rpy="0 0 0"/>
       <geometry>
-        <box size="${width} ${width} ${height1}"/>
-      </geometry>
-      <material name="orange"/>
-    </visual>
-    <inertial>
+        <box size="${base_width} ${base_depth} ${height1}"/>
+      </geometry>
+      <material name="purple"/>
+    </visual>
+    <!-- <inertial>
       <origin xyz="0 0 ${height1/2}" rpy="0 0 0"/>
       <mass value="${mass}"/>
@@ -36,12 +52,13 @@
         iyy="${mass / 12.0 * (height1*height1 + width*width)}" iyz="0.0"
         izz="${mass / 12.0 * (width*width + width*width)}"/>
-    </inertial>
+    </inertial> -->
   </link>
   <joint name="${prefix}shoulder" type="continuous">
-    <parent link="${prefix}base_link"/>
+    <parent link="${prefix}base_arm_link"/>
     <child link="${prefix}link1"/>
-    <origin xyz="0 ${width} ${height1 - axel_offset}" rpy="0 0 0"/>
-    <axis xyz="0 1 0"/>
-    <dynamics damping="0.7"/>
+    <origin xyz="0 0 ${height1}" rpy="0 0 0"/>
+    <axis xyz="0 1 0"/>
+    <dynamics damping="${damping}"/>
+    <dynamics friction="${friction}"/>
     <limit effort="100" velocity="1.0"/>
   </joint>
@@ -62,10 +79,10 @@
     </visual>
     <inertial>
-      <origin xyz="0 0 ${height2/2 - axel_offset}" rpy="0 0 0"/>
-      <mass value="${mass}"/>
-      <inertia
-        ixx="${mass / 12.0 * (width*width + height2*height2)}" ixy="0.0" ixz="0.0"
-        iyy="${mass / 12.0 * (height2*height2 + width*width)}" iyz="0.0"
-        izz="${mass / 12.0 * (width*width + width*width)}"/>
+      <origin xyz="-0.00009299 0.031668 0.45103767" rpy="0 0 0"/>
+      <mass value="1.57816"/>
+      <inertia
+        ixx="0.029411" ixy="0.00000451" ixz="-0.00001344"
+        iyy="0.027431" iyz="-0.0031087"
+        izz="0.0026470"/>
     </inertial>
   </link>
@@ -75,7 +92,11 @@
     <origin xyz="0 ${width} ${height2 - axel_offset*2}" rpy="0 0 0"/>
     <axis xyz="0 1 0"/>
-    <dynamics damping="0.7"/>
-    <limit effort="100" velocity="1.0"/>
-  </joint>
+    <dynamics damping="${damping}"/>
+    <dynamics friction="${friction}"/>
+    <limit effort="100" velocity="1.0"/>
+  </joint>
+  <xacro:property name="olnaExtraSizeX" value="0.044" />
+  <xacro:property name="olnaExtra2SizeY" value="0.10" />
+  <xacro:property name="olnaExtra2SizeZ" value="0.045" />
   <!-- Top Link -->
   <link name="${prefix}link2">
@@ -94,15 +115,154 @@
     </visual>
     <inertial>
-      <origin xyz="0 0 ${height3/2 - axel_offset}" rpy="0 0 0"/>
-      <mass value="${mass}"/>
-      <inertia
-        ixx="${mass / 12.0 * (width*width + height3*height3)}" ixy="0.0" ixz="0.0"
-        iyy="${mass / 12.0 * (height3*height3 + width*width)}" iyz="0.0"
-        izz="${mass / 12.0 * (width*width + width*width)}"/>
+      <origin xyz="-0.00002531 -0.029129 0.38624" rpy="0 0 0"/>
+      <mass value="0.71617"/>
+      <inertia
+        ixx="0.0216357" ixy="-0.00000056" ixz="0.00000268"
+        iyy="0.021156" iyz="0.0015021"
+        izz="0.00060628"/>
+    </inertial>
+  </link>
+  <joint name="${prefix}elbow_box_fix" type="fixed">
+    <parent link="${prefix}link2"/>
+    <child link="${prefix}link2_box"/>
+    <axis xyz="0 1 0"/>
+  </joint>
+  <link name="${prefix}link2_box">
+    <collision>
+      <origin xyz="0 ${-olnaExtra2SizeY/2 - width/2} ${height3 - olnaExtra2SizeZ}" rpy="0 0 0"/>
+      <geometry>
+        <box size="${olnaExtraSizeX} ${olnaExtra2SizeY} ${olnaExtra2SizeZ}"/>
+      </geometry>
+    </collision>
+    <visual>
+      <origin xyz="0 ${-olnaExtra2SizeY/2 - width/2} ${height3 - olnaExtra2SizeZ}" rpy="0 0 0"/>
+      <geometry>
+        <box size="${olnaExtraSizeX} ${olnaExtra2SizeY} ${olnaExtra2SizeZ}"/>
+      </geometry>
+      <material name="brown"/>
+    </visual>
+  </link>
+  <!-- Wrist 1 -->
+  <xacro:property name="wrist2SizeX" value="0.107" />
+  <xacro:property name="wrist2SizeY" value="0.053" />
+  <xacro:property name="wrist2SizeZ" value="0.05" />
+  <xacro:property name="wrist1AxelGap" value="0.007" />
+  <xacro:property name="wrist2AxelToRectTop" value="0.03" />
+  <joint name="${prefix}wrist1" type="continuous">
+    <parent link="${prefix}link2"/>
+    <child link="${prefix}wrist2"/>
+    <origin xyz="0 ${wrist1AxelGap + width/2} ${height3 - axel_offset*2}" rpy="0 0 0"/>
+    <axis xyz="0 1 0"/>
+    <dynamics damping="${damping}"/>
+    <dynamics friction="${friction}"/>
+    <limit effort="100" velocity="1.0"/>
+  </joint>
+  <link name="${prefix}wrist2">
+    <collision>
+      <origin xyz="${-wrist2AxelToRectTop + wrist2SizeX/2} ${wrist2SizeY/2} 0" rpy="0 0 0"/>
+      <geometry>
+        <box size="${wrist2SizeX} ${wrist2SizeY} ${wrist2SizeZ}"/>
+      </geometry>
+    </collision>
+    <visual>
+      <origin xyz="${-wrist2AxelToRectTop + wrist2SizeX/2} ${wrist2SizeY/2} 0" rpy="0 0 0"/>
+      <geometry>
+        <box size="${wrist2SizeX} ${wrist2SizeY} ${wrist2SizeZ}"/>
+      </geometry>
+      <material name="green"/>
+    </visual>
+    <inertial>
+      <origin xyz="0.011680 0.024878 -0.0007064" rpy="0 0 0"/>
+      <mass value="0.49788"/>
+      <inertia
+        ixx="0.00014917" ixy="-0.00002443" ixz="0.00000086"
+        iyy="0.00050396" iyz="0.00000032"
+        izz="0.00053155"/>
+    </inertial>
+  </link>
+  <!-- Wrist 3 -->
+  <xacro:property name="wrist3SizeX" value="0.053" />
+  <xacro:property name="wrist3SizeY" value="0.05" />
+  <xacro:property name="wrist3SizeZ" value="0.107" />
+<!--  distance between boxes  -->
+  <xacro:property name="wrist2AxelGap" value="0.002" />
+  <xacro:property name="wrist3AxelToRectTop" value="0.025" />
+  <joint name="${prefix}wrist2_joint" type="continuous">
+    <parent link="${prefix}wrist2"/>
+    <child link="${prefix}wrist3"/>
+<!-- in parent coords -->
+    <origin xyz="${-wrist2AxelToRectTop} ${wrist2SizeY/2} ${0}" rpy="0 0 0"/>
+    <axis xyz="1 0 0"/>
+    <dynamics damping="${damping}"/>
+    <dynamics friction="${friction}"/>
+    <limit effort="100" velocity="1.0"/>
+  </joint>
+  <link name="${prefix}wrist3">
+    <collision>
+      <origin xyz="${-wrist2AxelGap - wrist3SizeX/2} ${0} ${-wrist3SizeZ/2 + wrist3AxelToRectTop}" rpy="0 0 0"/>
+      <geometry>
+        <box size="${wrist3SizeX} ${wrist3SizeY} ${wrist3SizeZ}"/>
+      </geometry>
+    </collision>
+    <visual>
+      <origin xyz="${-wrist2AxelGap - wrist3SizeX/2} ${0} ${-wrist3SizeZ/2 + wrist3AxelToRectTop}" rpy="0 0 0"/>
+      <geometry>
+        <box size="${wrist3SizeX} ${wrist3SizeY} ${wrist3SizeZ}"/>
+      </geometry>
+      <material name="blue"/>
+    </visual>
+    <!-- TODO URC-442: add in a mass and moment of inertia for Wrist3 -->
+    <inertial>
+      <origin xyz="-0.026878 -0.00007064 0.011680" rpy="0 0 0"/>
+      <mass value="0.49788"/>
+      <inertia
+        ixx="0.00050396" ixy="-0.00000032" ixz="-0.00002443"
+        iyy="0.00053155" iyz="-0.00000086"
+        izz="0.00014917"/>
+    </inertial>
+  </link>
+<!-- end effector -->
+  <xacro:property name="endeSizeX" value="0.03" />
+  <xacro:property name="endeSizeY" value="0.11" />
+  <xacro:property name="endeSizeZ" value="0.24" />
+<!--  distance between boxes  -->
+  <xacro:property name="wrist3AxelGap" value="0.01" />
+  <!-- <xacro:property name="endeAxelToRectTop" value="0.01" />  -->
+  <joint name="${prefix}wrist3_joint" type="continuous">
+    <parent link="${prefix}wrist3"/>
+    <child link="${prefix}endEffector"/>
+<!-- in parent coords -->
+    <origin xyz="${-wrist3SizeX/2} 0 ${0}" rpy="0 0 0"/>
+    <axis xyz="0 0 1"/>
+    <dynamics damping="${damping}"/>
+    <dynamics friction="${friction}"/>
+    <limit effort="100" velocity="1.0"/>
+  </joint>
+  <link name="${prefix}endEffector">
+    <collision>
+      <origin xyz="0 0 ${endeSizeZ/2 + wrist3AxelToRectTop + wrist3AxelGap}" rpy="0 0 0"/>
+      <geometry>
+        <box size="${endeSizeX} ${endeSizeY} ${endeSizeZ}"/>
+      </geometry>
+    </collision>
+    <visual>
+      <origin xyz="0 0 ${endeSizeZ/2 + wrist3AxelToRectTop + wrist3AxelGap}" rpy="0 0 0"/>
+      <geometry>
+        <box size="${endeSizeX} ${endeSizeY} ${endeSizeZ}"/>
+      </geometry>
+      <material name="white"/>
+    </visual>
+    <inertial>
+      <origin xyz="-0.038139 0.016827 -0.052402" rpy="0 0 0"/>
+      <mass value="0.59465"/>
+      <inertia
+        ixx="0.00061465" ixy="0.00023266" ixz="0.00017509"
+        iyy="0.00117167" iyz="-0.00007772"
+        izz="0.0011538"/>
     </inertial>
   </link>
   <joint name="${prefix}tool_joint" type="fixed">
-    <origin xyz="0 0 1" rpy="0 0 0" />
-    <parent link="${prefix}link2"/>
+    <origin xyz="0 0 ${endeSizeZ + wrist3AxelToRectTop + wrist3AxelGap}" rpy="0 0 0" />
+    <parent link="${prefix}endEffector"/>
     <child link="${prefix}tool_link" />
   </joint>
